File: mainbrd3.kicad_sch (KiCad schematic)
At the start: 0 parts

Commit message: Autosave
Other:
- added sheet ETH (ETH.kicad_sch)
- added sheet MCU (untitled.kicad_sch)
- added sheet sheet 3 (sheet3.kicad_sch)
Changed lines of the file:
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@@
 (kicad_sch
-	(version 20260306)
+	(version 20231120)
 	(generator "eeschema")
-	(generator_version "10.0")
-	(paper "A4")
+	(generator_version "8.0")
+	(paper "A3")
+	(sheet
+		(at 38.1 30.48)
+		(size 63.5 80.01)
+		(fields_autoplaced yes)
+		(stroke
+			(width 0.1524)
+			(type solid)
+		)
+		(fill
+			(color 0 0 0 0.0000)
+		)
+		(property "Sheetname" "MCU"
+			(at 38.1 29.7684 0)
+			(effects
+				(font
+					(size 1.27 1.27)
+				)
+				(justify left bottom)
+			)
+		)
+		(property "Sheetfile" "untitled.kicad_sch"
+			(at 38.1 111.0746 0)
+			(effects
+				(font
+					(size 1.27 1.27)
+				)
+				(justify left top)
+			)
+		)
+		(instances
+			(project "mainbrd1"
+				(path "/89e0f049-91ab-4c37-b514-d5ee0e775d39"
+					(page "2")
+				)
+			)
+		)
+	)
+	(sheet
+		(at 187.96 33.02)
+		(size 59.69 78.74)
+		(fields_autoplaced yes)
+		(stroke
+			(width 0.1524)
+			(type solid)
+		)
+		(fill
+			(color 0 0 0 0.0000)
+		)
+		(property "Sheetname" "sheet 3"
+			(at 187.96 32.3084 0)
+			(effects
+				(font
+					(size 1.27 1.27)
+				)
+				(justify left bottom)
+			)
+		)
+		(property "Sheetfile" "sheet3.kicad_sch"
+			(at 187.96 112.3446 0)
+			(effects
+				(font
+					(size 1.27 1.27)
+				)
+				(justify left top)
+			)
+		)
+		(instances
+			(project "mainbrd1"
+				(path "/89e0f049-91ab-4c37-b514-d5ee0e775d39"
+					(page "4")
+				)
+			)
+		)
+	)
+	(sheet
+		(at 114.3 30.48)
+		(size 66.04 80.01)
+		(fields_autoplaced yes)
+		(stroke
+			(width 0.1524)
+			(type solid)
+		)
+		(fill
+			(color 0 0 0 0.0000)
+		)
+		(property "Sheetname" "ETH"
+			(at 114.3 29.7684 0)
+			(effects
+				(font
+					(size 1.27 1.27)
+				)
+				(justify left bottom)
+			)
+		)
+		(property "Sheetfile" "ETH.kicad_sch"
+			(at 114.3 111.0746 0)
+			(effects
+				(font
+					(size 1.27 1.27)
+				)
+				(justify left top)
+			)
+		)
+		(instances
+			(project "mainbrd1"
+				(path "/89e0f049-91ab-4c37-b514-d5ee0e775d39"
+					(page "3")
+				)
+			)
+		)
+	)
 	(sheet_instances
 		(path "/"
@@
 		)
 	)
-	(embedded_fonts no)
 )

Commit message: SCH Save: 2 files changed mainbrd3.kicad_pro 6/0/1 mainbrd3.kicad_sch 25/0/9
Other:
- sheet sheet 3 renamed rs485
Changed lines of the file:
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@@
 (kicad_sch
-	(version 20231120)
+	(version 20260306)
 	(generator "eeschema")
-	(generator_version "8.0")
+	(generator_version "10.0")
 	(paper "A3")
 	(sheet
 		(at 38.1 30.48)
 		(size 63.5 80.01)
+		(exclude_from_sim no)
+		(in_bom yes)
+		(on_board yes)
+		(dnp no)
 		(fields_autoplaced yes)
 		(stroke
@@
 		)
 		(fill
-			(color 0 0 0 0.0000)
+			(color 0 0 0 0)
 		)
 		(property "Sheetname" "MCU"
 			(at 38.1 29.7684 0)
+			(show_name no)
+			(do_not_autoplace no)
 			(effects
 				(font
@@
 		(property "Sheetfile" "untitled.kicad_sch"
 			(at 38.1 111.0746 0)
+			(show_name no)
+			(do_not_autoplace no)
 			(effects
 				(font
@@
 		)
 		(instances
-			(project "mainbrd1"
+			(project "mainbrd3"
 				(path "/89e0f049-91ab-4c37-b514-d5ee0e775d39"
 					(page "2")
@@
 		(at 187.96 33.02)
 		(size 59.69 78.74)
+		(exclude_from_sim no)
+		(in_bom yes)
+		(on_board yes)
+		(dnp no)
 		(fields_autoplaced yes)
 		(stroke
@@
 		)
 		(fill
-			(color 0 0 0 0.0000)
+			(color 0 0 0 0)
 		)
-		(property "Sheetname" "sheet 3"
+		(property "Sheetname" "rs485"
 			(at 187.96 32.3084 0)
+			(show_name no)
+			(do_not_autoplace no)
 			(effects
 				(font
@@
 		(property "Sheetfile" "sheet3.kicad_sch"
 			(at 187.96 112.3446 0)
+			(show_name no)
+			(do_not_autoplace no)
 			(effects
 				(font
@@
 		)
 		(instances
-			(project "mainbrd1"
+			(project "mainbrd3"
 				(path "/89e0f049-91ab-4c37-b514-d5ee0e775d39"
 					(page "4")
@@
 		(at 114.3 30.48)
 		(size 66.04 80.01)
+		(exclude_from_sim no)
+		(in_bom yes)
+		(on_board yes)
+		(dnp no)
 		(fields_autoplaced yes)
 		(stroke
@@
 		)
 		(fill
-			(color 0 0 0 0.0000)
+			(color 0 0 0 0)
 		)
 		(property "Sheetname" "ETH"
 			(at 114.3 29.7684 0)
+			(show_name no)
+			(do_not_autoplace no)
 			(effects
 				(font
@@
 		(property "Sheetfile" "ETH.kicad_sch"
 			(at 114.3 111.0746 0)
+			(show_name no)
+			(do_not_autoplace no)
 			(effects
 				(font
@@
 		)
 		(instances
-			(project "mainbrd1"
+			(project "mainbrd3"
 				(path "/89e0f049-91ab-4c37-b514-d5ee0e775d39"
 					(page "3")
@@
 		)
 	)
+	(embedded_fonts no)
 )
