File: mainbrd3.kicad_pcb (KiCad board)
At the start: 4 copper layers, 112 parts, among them J1 Conn_01x04_Pin, J10 Conn_01x03_Pin, J2 USB_B_Micro, J3 Conn_01x02_Pin, J4 Conn_01x02_Pin, J5 https://abracon.com/Magnetics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, J6 Screw_Terminal_01x02, J7 Screw_Terminal_01x02, J8 Screw_Terminal_01x02, J9 Screw_Terminal_01x02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

Commit message: PCB Save: 2 files changed mainbrd3.kicad_pcb 0/0/469 mainbrd3.kicad_prl 0/0/1
Parts:
- moved J2 130.1 mm to (163.9, 65.5), turned to 180 degrees
- moved J5 64.9 mm to (193.0, 80.0), turned to 180 degrees
- moved U5 56.1 mm to (111.8, 70.5)
- moved U3 52.7 mm to (187.0, 90.2)
- moved U1 14.4 mm to (159.5, 95.0), turned to 90 degrees
Connections:
- J10 pad 1: /MCU/UART8_RX -> /MCU/UART3_TX
- J10 pad 2: /MCU/UART8_TX -> /MCU/UART3_RX
- U1 pad 102: UART4_DIR -> unconnected-(U1-PA10-Pad102)
- U1 pad 103: UART4_RX -> D-
- U1 pad 104: UART4_TX -> D+
- U1 pad 110: unconnected-(U1-PA15-Pad110) -> UART4_DIR
- U1 pad 111: unconnected-(U1-PC10-Pad111) -> UART4_TX
- U1 pad 112: unconnected-(U1-PC11-Pad112) -> UART4_RX
- U1 pad 117: UART5_DIR -> unconnected-(U1-PD3-Pad117)
- U1 pad 141: /MCU/UART8_RX -> unconnected-(U1-PE0-Pad141)
- U1 pad 142: /MCU/UART8_TX -> unconnected-(U1-PE1-Pad142)
- U1 pad 75: D- -> unconnected-(U1-PB14-Pad75)
- U1 pad 76: D+ -> unconnected-(U1-PB15-Pad76)
- U1 pad 77: unconnected-(U1-PD8-Pad77) -> /MCU/UART3_TX
- U1 pad 78: unconnected-(U1-PD9-Pad78) -> /MCU/UART3_RX
- U1 pad 98: unconnected-(U1-PC8-Pad98) -> UART5_DIR

Commit message: PCB Save: 2 files changed mainbrd3.kicad_pcb 40/0/0 mainbrd3.kicad_pro 17/0/1
Other:
- board outline added: 100 x 72 mm
Changed lines of the file:
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@@
 		)
+	)
+	(gr_line
+		(start 103 59)
+		(end 103 131)
+		(stroke
+			(width 0.05)
+			(type default)
+		)
+		(layer "Edge.Cuts")
+	)
+	(gr_line
+		(start 103 59)
+		(end 203 59)
+		(stroke
+			(width 0.05)
+			(type default)
+		)
+		(layer "Edge.Cuts")
+	)
+	(gr_line
+		(start 103 131)
+		(end 203 131)
+		(stroke
+			(width 0.05)
+			(type default)
+		)
+		(layer "Edge.Cuts")
+	)
+	(gr_line
+		(start 203 131)
+		(end 203 59)
+		(stroke
+			(width 0.05)
+			(type default)
+		)
+		(layer "Edge.Cuts")
 	)
 	(embedded_fonts no)

Commit message: PCB Save: 3 files changed mainbrd3.kicad_pcb 861/0/135 mainbrd3.kicad_prl 13/0/4 ~mainbrd3.kicad_pro.lck 1/0/0
Parts:
- moved C7 119.7 mm to (172.5, 103.0)
- moved C6 119.2 mm to (172.5, 97.0)
- moved C5 119.0 mm to (172.5, 92.0)
- moved C4 118.9 mm to (172.5, 86.0)
- moved C8 112.1 mm to (165.0, 108.0), turned to -90 degrees
- moved R21 111.5 mm to (199.0, 65.0)
- moved C3 109.5 mm to (163.0, 82.0), turned to 90 degrees
- moved C9 105.8 mm to (159.0, 108.0), turned to -90 degrees
- moved C28 102.8 mm to (181.5, 90.0)
- moved C10 99.5 mm to (153.0, 108.0), turned to -90 degrees
- moved C13 95.8 mm to (132.2, 97.0)
- moved C34 91.9 mm to (151.0, 82.0), turned to 90 degrees
- moved C11 91.9 mm to (146.5, 104.0), turned to 180 degrees
- moved C12 90.5 mm to (146.5, 97.0), turned to 180 degrees
- moved R22 89.6 mm to (176.0, 65.0)
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Routing:
- added copper zone on In2.Cu, net +3V3
- added copper zone on In1.Cu, net GND

Commit message: PCB Save: 2 files changed mainbrd3.kicad_pcb 1188/0/386 mainbrd3.kicad_prl 0/0/2
Parts:
- moved C13 10.2 mm to (142.0, 94.0), turned to 180 degrees
- moved C5 1.00 mm to (172.5, 91.0), turned to -90 degrees
- moved C6 0.52 mm to (172.5, 96.5), turned to -90 degrees
- turned C12 to 90 degrees
- turned C3 to 0 degrees
- turned C34 to 0 degrees
- turned C7 to -90 degrees
- turned C8 to 0 degrees
- turned C9 to 180 degrees
Routing:
- net +3V3: track 0.00 -> 40.3 mm, vias 0 -> 10
- net GND: track 0.00 -> 37.9 mm, vias 0 -> 13

Commit message: PCB Save: 3 files changed mainbrd3.kicad_pcb 748/0/2692 mainbrd3.kicad_prl 0/0/2 mainbrd3.kicad_pro 0/0/1
Parts:
- removed D2: MBR0580, Diode_SMD:D_SOD-123
- removed F2: Fuse, Fuse:Fuse_1206_3216Metric
- C19, R1, R2: moved to B.Cu
- moved U2 93.1 mm to (119.2, 74.6)
- moved JP1 92.1 mm to (129.4, 71.4), turned to 180 degrees
- moved C20 83.4 mm to (128.9, 74.7)
- moved R2 78.4 mm to (116.1, 72.3), turned to 90 degrees
- moved R1 77.8 mm to (114.6, 72.8)
- moved J6 75.1 mm to (122.5, 41.2)
- moved C19 73.0 mm to (116.9, 77.1), turned to -90 degrees
- moved C14 71.4 mm to (113.6, 76.2), turned to 180 degrees
- moved J9 71.0 mm to (114.9, 64.0)
- moved L1 67.5 mm to (123.4, 73.1)
- moved D1 58.5 mm to (113.5, 73.6), turned to 180 degrees
- moved R16 56.5 mm to (78.5, 100.0)
- moved R20 56.5 mm to (80.9, 94.1)
- moved R9 56.5 mm to (75.5, 100.0)
- moved C21 56.5 mm to (75.5, 106.0)
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Connections:
- J5 pad 9: +V_POE -> unconnected-(J5-V+-Pad9)
Routing:
- net /MCU/3v3smps: track 0.00 -> 10.9 mm
- net Net-(D1-K): track 0.00 -> 5.11 mm, vias 0 -> 1
- net Net-(U2-EN/UVLO): track 0.00 -> 4.98 mm, vias 0 -> 1
- net GND: track 37.9 -> 41.6 mm, vias 13 -> 25
- net Net-(U2-VCC): track 0.00 -> 2.36 mm, vias 0 -> 1
- net +3V3: vias 10 -> 22
- added copper zone on F.Cu, net +12V
- added copper zone on F.Cu, net +3V3
- added copper zone on F.Cu, net /MCU/3v3smps
- added copper zone on F.Cu, net /MCU/sw-3v3
- added copper zone on B.Cu, net Earth
- added copper zone on F.Cu, net GND
- added copper zone on F.Cu, net Net-(D1-A)
- added copper zone on F.Cu, net Net-(D1-K)

Commit message: PCB Save: 2 files changed mainbrd3.kicad_pcb 79/0/261 mainbrd3.kicad_prl 0/0/2
Routing:
- net GND: vias 25 -> 29
Changed lines of the file:
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@@
+	)
+	(via
+		(at 131 76.4)
+		(size 0.6)
+		(drill 0.3)
+		(layers "F.Cu" "B.Cu")
+		(free yes)
+		(net "GND")
 	)
 	(via
@@
 	)
 	(via
+		(at 131 74.6)
+		(size 0.6)
+		(drill 0.3)
+		(layers "F.Cu" "B.Cu")
+		(free yes)
+		(net "GND")
+	)
+	(via
 		(at 151.48 81.02)
 		(size 0.6)
@@
 		(drill 0.3)
 		(layers "F.Cu" "B.Cu")
+		(net "GND")
+	)
+	(via
+		(at 131 75.5)
+		(size 0.6)
+		(drill 0.3)
+		(layers "F.Cu" "B.Cu")
+		(free yes)
 		(net "GND")
 	)
@@
 		(size 0.6)
 		(drill 0.3)
+		(layers "F.Cu" "B.Cu")
+		(free yes)
+		(net "GND")
+	)
+	(via
+		(at 129.7 76.4)
+		(size 0.6)
+		(drill 0.3)

Commit message: PCB Save: 3 files changed mainbrd3.kicad_pcb 0/38/838 mainbrd3.kicad_prl 0/0/2 mainbrd3.kicad_pro 0/0/1
Parts:
- moved C19 3.10 mm to (116.9, 80.2)
- moved D1 3.10 mm to (113.5, 76.7)
- moved F1 3.10 mm to (113.5, 74.2)
- moved L1 3.10 mm to (123.4, 76.2)
- moved R1 3.10 mm to (114.6, 75.9)
- moved U2 3.10 mm to (119.2, 77.7)
- moved C14 3.10 mm to (113.6, 79.3)
- moved C20 3.10 mm to (128.9, 77.8)
- moved JP1 3.10 mm to (129.4, 74.5)
- moved R2 3.10 mm to (116.1, 75.4)

Commit message: PCB Save: 3 files changed mainbrd3.kicad_pcb 627/0/725 mainbrd3.kicad_prl 0/0/1 mainbrd3.kicad_pro 0/0/1
Parts:
- C32: moved to B.Cu
- moved U8 104.9 mm to (138.1, 74.0), turned to 180 degrees
- moved C32 84.4 mm to (143.1, 74.1), turned to -90 degrees
- moved J2 10.7 mm to (153.2, 62.8)
Routing:
- net +5VUSB: track 0.00 -> 2.22 mm, vias 0 -> 7
- net GND: track 41.6 -> 43.2 mm, vias 29 -> 41
- added copper zone on B.Cu, net +5VUSB
- added copper zone on F.Cu, net +5VUSB
- added copper zone on F.Cu, net /MCU/3v3_usb
