File: mainbrd3.kicad_pcb (KiCad board)
At the start: 4 copper layers, 100 x 72 mm, 110 parts, among them J1 Conn_01x04_Pin, J10 Conn_01x03_Pin, J2 USB_B_Micro, J3 Conn_01x02_Pin, J4 Conn_01x02_Pin, J5 https://abracon.com/Magnetics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, J6 Screw_Terminal_01x02, J7 Screw_Terminal_01x02, J8 Screw_Terminal_01x02, J9 Screw_Terminal_01x02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

Commit message: PCB Save: 1 files changed mainbrd3.kicad_pcb 0/1609/14497
Parts:
- C10, C3, C4, C8, C9, R14, R15, R16, R19: moved to B.Cu
- moved C26 122.5 mm to (199.2, 87.8)
- moved C25 122.5 mm to (199.2, 85.9)
- moved C24 115.9 mm to (188.5, 84.1), turned to 180 degrees
- moved C30 110.0 mm to (185.7, 81.8)
- moved R18 31.7 mm to (207.9, 105.1)
- moved R17 17.2 mm to (207.8, 97.1)
- moved C9 13.6 mm to (158.4, 99.9)
- moved C8 13.2 mm to (165.1, 99.9)
- moved C4 12.3 mm to (170.0, 82.6)
- moved C10 11.5 mm to (152.9, 102.4)
- moved R10 10.9 mm to (205.2, 101.8)
- moved C6 10.3 mm to (172.3, 93.1)
- moved R11 10.3 mm to (173.7, 97.0)
- moved R12 10.3 mm to (173.7, 95.8)
- moved U1 10.3 mm to (159.2, 91.7)
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Routing:
- net NRST: track 51.9 -> 0.00 mm, vias 2 -> 0
- net Net-(U3-~{INT}/REFCLKO): track 45.0 -> 0.00 mm, vias 4 -> 0
- net ETH_MDC: track 40.1 -> 0.00 mm, vias 2 -> 0
- net +3V3_ethtxrx: track 29.4 -> 67.4 mm
- net ETH_MDIO: track 35.1 -> 0.00 mm, vias 3 -> 0
- net I2C1_SDA: track 37.0 -> 3.11 mm, vias 2 -> 1
- net I2C1_SCL: track 35.6 -> 2.35 mm, vias 2 -> 1
- net Net-(U3-CRS_DV/MODE2): track 26.7 -> 0.00 mm, vias 3 -> 0
- net Net-(U3-RXD0/MODE0): track 25.1 -> 0.00 mm, vias 3 -> 0
- net ETH_TXD0: track 34.9 -> 20.8 mm
- net ETH_TXD1: track 37.1 -> 23.9 mm
- net Net-(U3-RXER/PHYAD0): track 12.3 -> 0.00 mm, vias 2 -> 0
- net D-: track 27.0 -> 16.7 mm
- net D+: track 26.9 -> 16.7 mm
- net +3V3: track 59.9 -> 53.6 mm, vias 37 -> 38
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- removed copper zone on F.Cu, net +3V3_ethtxrx
- removed copper zone on In2.Cu, net +3V3_ethtxrx

Commit message: PCB Save: 1 files changed mainbrd3.kicad_pcb 884/0/1505
Parts:
- C21, C22, C23, R10, R17: moved to B.Cu
- R18: moved to F.Cu
- moved C23 116.2 mm to (191.0, 91.8), turned to 180 degrees
- moved C21 113.6 mm to (188.6, 91.4), turned to 180 degrees
- moved C22 107.8 mm to (189.1, 88.8), turned to 90 degrees
- moved R10 15.8 mm to (193.9, 90.8), turned to 0 degrees
- moved R18 14.3 mm to (195.6, 97.8), turned to 90 degrees
- moved R17 13.7 mm to (194.4, 94.3), turned to 90 degrees
- moved R19 3.71 mm to (195.6, 94.3)
- moved R14 2.38 mm to (192.0, 94.3)
- moved R16 1.50 mm to (193.2, 94.3)
- moved R15 0.89 mm to (190.9, 94.3)
Routing:
- net NRST: track 0.00 -> 49.1 mm, vias 0 -> 2
- net ETH_MDC: track 0.00 -> 45.4 mm, vias 0 -> 2
- net ETH_MDIO: track 0.00 -> 42.0 mm, vias 0 -> 1
- net ETH_REF_CLK: track 0.00 -> 33.2 mm
- net Net-(U3-CRS_DV/MODE2): track 0.00 -> 26.6 mm, vias 0 -> 1
- net Net-(U3-RXD0/MODE0): track 0.00 -> 25.1 mm, vias 0 -> 1
- net Net-(U3-~{INT}/REFCLKO): track 0.00 -> 12.0 mm, vias 0 -> 1
- net GND: track 60.2 -> 71.1 mm
- net Net-(U3-VDDCR): track 0.00 -> 4.61 mm, vias 0 -> 1
- net ETH_TXD0: track 20.8 -> 25.2 mm
- net ETH_TXD1: track 23.9 -> 28.0 mm
- net Net-(U3-RXER/PHYAD0): track 0.00 -> 3.12 mm, vias 0 -> 1
- net +3V3: track 53.6 -> 54.9 mm
- net +3V3_ethtxrx: track 67.4 -> 68.4 mm
- net Net-(U3-RXD1/MODE1): track 23.3 -> 24.0 mm

Commit message: PCB Save: 1 files changed mainbrd3.kicad_pcb 0/8/243
Parts:
- moved D3 14.2 mm to (162.5, 113.8)
- moved R34 14.2 mm to (162.5, 117.5)
- moved U6 14.2 mm to (162.6, 110.8)
- moved R29 14.2 mm to (158.2, 111.6)
- moved R31 14.2 mm to (158.2, 109.4)
- moved R30 14.2 mm to (158.2, 110.5)
- moved R32 14.2 mm to (163.7, 116.3)
- moved R33 14.2 mm to (161.4, 116.3)
- moved R35 13.9 mm to (173.6, 111.5)
- moved R36 13.9 mm to (173.6, 110.4)
- moved R38 13.9 mm to (176.7, 116.0)
- moved R39 13.9 mm to (179.0, 116.0)
- moved R40 13.9 mm to (177.8, 117.2)
- moved D4 13.9 mm to (177.9, 113.5)
- moved R37 13.9 mm to (173.6, 109.3)
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Routing:
- net ETH_REF_CLK: track 33.2 -> 32.1 mm
- net ETH_MDIO: track 42.0 -> 41.2 mm

Commit message: PCB Save: 1 files changed mainbrd3.kicad_pcb 1980/0/2540
Parts:
- moved Y1 136.9 mm to (161.8, 108.0)
- moved H3 132.8 mm to (199.6, 62.1)
- moved C2 114.2 mm to (165.0, 107.2)
- moved C1 108.9 mm to (158.6, 109.0), turned to 180 degrees
- moved C17 81.4 mm to (135.8, 107.8)
- moved C15 64.6 mm to (117.1, 112.3)
- moved C18 64.6 mm to (120.0, 104.4)
- moved C33 64.6 mm to (120.0, 108.4)
- moved C16 64.6 mm to (116.8, 115.6)
- moved D3 13.3 mm to (175.8, 113.8)
- moved D4 13.3 mm to (191.2, 113.5)
- moved J7 13.3 mm to (173.0, 126.9)
- moved J8 13.3 mm to (187.9, 127.0)
- moved R29 13.3 mm to (171.5, 111.6)
- moved R30 13.3 mm to (171.5, 110.5)
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Connections:
- J2 pad SH: Earth -> (no net)
- J5 pad 9: unconnected-(J5-V+-Pad9) -> +V_POE
- J7 pad 1: Net-(D3-A1) -> Net-(D3-A2)
- J7 pad 2: Net-(D3-A2) -> Net-(D3-A1)
- J8 pad 1: Net-(D4-A1) -> Net-(D4-A2)
- J8 pad 2: Net-(D4-A2) -> Net-(D4-A1)
Routing:
- net UART4_DIR: track 5.89 -> 65.0 mm, vias 0 -> 4
- net UART4_RX: track 7.72 -> 64.1 mm, vias 0 -> 3
- net UART4_TX: track 3.44 -> 55.9 mm, vias 0 -> 4
- net UART5_RX: track 7.88 -> 51.2 mm, vias 0 -> 2
- net UART5_DIR: track 5.96 -> 48.4 mm, vias 0 -> 2
- net I2C1_SDA: track 3.11 -> 43.0 mm, vias 1 -> 2
- net I2C1_SCL: track 2.35 -> 41.8 mm, vias 1 -> 2
- net UART5_TX: track 2.40 -> 41.4 mm, vias 0 -> 2
- net Net-(D4-A2): track 6.94 -> 17.9 mm
- net Net-(D3-A2): track 6.98 -> 17.4 mm
- net Net-(D4-A1): track 6.95 -> 17.3 mm
- net Net-(D3-A1): track 6.86 -> 17.0 mm
- net /MCU/RCC_OSC_IN: track 0.00 -> 8.72 mm
- net GND: track 71.1 -> 78.5 mm, vias 61 -> 65
- net /MCU/RCC_OSC_OUT: track 0.00 -> 6.82 mm
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
Commit message: PCB Save: 2 files changed mainbrd3.kicad_pcb 402/0/1099 mainbrd3.kicad_prl 0/0/1
Parts:
- moved L3 146.0 mm to (167.3, 105.0), turned to 180 degrees
- moved C15 52.9 mm to (169.6, 105.7), turned to -90 degrees
- moved C17 29.4 mm to (165.0, 104.5), turned to 90 degrees
Routing:
- net +3V3VADC: track 0.00 -> 3.97 mm
- net GND: track 78.5 -> 81.2 mm, vias 65 -> 66
- net +3V3: track 56.0 -> 58.4 mm, vias 38 -> 39
- net ETH_REF_CLK: track 34.9 -> 32.5 mm
- net UART5_TX: track 41.4 -> 43.0 mm
- net UART5_DIR: track 48.4 -> 49.3 mm
- added copper zone on B.Cu, net +3V3VADC

Commit message: PCB Save: 1 files changed mainbrd3.kicad_pcb 95/0/467
Parts:
- moved C18 47.9 mm to (167.8, 106.6)
- moved C15 0.20 mm to (169.8, 105.7)
Routing:
- net GND: track 81.2 -> 85.6 mm
- net +3V3VADC: track 3.97 -> 6.23 mm
Changed lines of the file:
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@@
 	(footprint "Capacitor_SMD:C_0402_1005Metric"
 		(layer "F.Cu")
-		(at 169.6 105.7 -90)
+		(at 169.8 105.7 -90)
 		(descr "Capacitor SMD 0402 (1005 Metric), square (rectangular) end terminal, IPC-7351 nominal, (Body size source: IPC-SM-782 page 76, https://www.pcb-3d.com/wordpress/wp-content/uploads/ipc-sm-782a_amendment_1_and_2.pdf)")
 		(tags "capacitor")
@@
 	(footprint "Capacitor_SMD:C_0402_1005Metric"
 		(layer "F.Cu")
-		(at 119.95 104.42)
+		(at 167.82 106.6)
 		(descr "Capacitor SMD 0402 (1005 Metric), square (rectangular) end terminal, IPC-7351 nominal, (Body size source: IPC-SM-782 page 76, https://www.pcb-3d.com/wordpress/wp-content/uploads/ipc-sm-782a_amendment_1_and_2.pdf)")
 		(tags "capacitor")
@@
 	)
 	(segment
-		(start 169.6 106.18)
-		(end 169.6 107.4)
-		(width 0.3)
-		(layer "F.Cu")
-		(net "GND")
-	)
-	(segment
 		(start 157.5 100.9)
 		(end 157.6 100.9)
@@
 	)
 	(segment
+		(start 170.8 106.2)
+		(end 170.78 106.18)
+		(width 0.3)
+		(layer "F.Cu")
+		(net "GND")
+	)
+	(segment
 		(start 187.81 113.06875)
 		(end 189.22 113.06875)
@@
 	)
 	(segment
+		(start 162.9 108.85)
+		(end 163.95 108.85)
+		(width 0.3)
+		(layer "F.Cu")
+		(net "GND")
+	)
+	(segment
 		(start 150.95 81.0375)
 		(end 150.95 79.45)
@@
 	)
 	(segment
+		(start 163.95 108.85)
+		(end 164.2 109.1)
+		(width 0.3)
+		(layer "F.Cu")
+		(net "GND")
+	)
+	(segment
 		(start 165.48 107.2)
 		(end 165.48 108.72)
@@
 	)
 	(segment
+		(start 169.38 106.6)
+		(end 169.8 106.18)
+		(width 0.5)
+		(layer "F.Cu")
+		(net "GND")
+	)
+	(segment
 		(start 199.68 85.9)
 		(end 200.6 85.9)
@@
 	)
 	(segment
+		(start 159.25 107.15)
+		(end 159.2 107.1)
+		(width 0.3)
+		(layer "F.Cu")
+		(net "GND")
+	)
+	(segment
 		(start 171.35 88.45)
 		(end 169.8625 88.45)
@@
 	)
 	(segment
+		(start 168.3 106.6)
+		(end 169.38 106.6)
+		(width 0.5)
+		(layer "F.Cu")
+		(net "GND")
+	)
+	(segment
 		(start 173.8375 113.35625)
 		(end 173.9625 113.23125)
@@
 	)
 	(segment
+		(start 170.78 106.18)
+		(end 169.8 106.18)
+		(width 0.3)
+		(layer "F.Cu")
+		(net "GND")
+	)
+	(segment
 		(start 169.735 75.775)
 		(end 168.405 75.775)
@@
 	)
 	(segment
+		(start 160.7 107.15)
+		(end 159.25 107.15)
+		(width 0.3)
+		(layer "F.Cu")
+		(net "GND")
+	)
+	(segment
 		(start 192.83 115.96875)
 		(end 192.83 117.14875)
@@
 	)
 	(via
-		(at 169.6 107.4)
+		(at 170.8 106.2)
 		(size 0.6)
 		(drill 0.3)
@@
 	)
 	(segment
-		(start 168.5825 105.22)
-		(end 168.3625 105)
-		(width 0.3)
-		(layer "F.Cu")
-		(net "+3V3")
-	)
-	(segment
 		(start 171.5075 99.0925)
 		(end 172.4 99.0925)
@@
 	)
 	(segment
+		(start 168.5825 105.22)
+		(end 168.3625 105)
+		(width 0.5)
+		(layer "F.Cu")
+		(net "+3V3")
+	)
+	(segment
 		(start 147.155 93.95)
 		(end 147.0525 94.0525)
@@
 	)
 	(segment
-		(start 169.6 105.22)
-		(end 168.5825 105.22)
-		(width 0.3)
-		(layer "F.Cu")
-		(net "+3V3")
-	)
-	(segment
 		(start 150.45 81.0375)
 		(end 149.94 80.5275)
@@
 	)
 	(segment
+		(start 169.8 105.22)
+		(end 168.5825 105.22)
+		(width 0.5)
+		(layer "F.Cu")
+		(net "+3V3")
+	)
+	(segment
 		(start 193.01 111.16875)
 		(end 193.08 111.23875)
@@
 	)
 	(segment
+		(start 166.2375 105.8375)
+		(end 166.2375 105)
+		(width 0.5)
+		(layer "F.Cu")
+		(net "+3V3VADC")
+	)
+	(segment
+		(start 167.34 106.6)
+		(end 167 106.6)
+		(width 0.5)
+		(layer "F.Cu")
+		(net "+3V3VADC")
+	)
+	(segment
 		(start 166.2375 102.55)
 		(end 166.05 102.3625)
@@
 		(width 0.5)
 		(layer "F.Cu")
+		(net "+3V3VADC")
+	)
+	(segment
+		(start 167 106.6)
+		(end 166.2375 105.8375)
+		(width 0.5)
+		(layer "F.Cu")

Commit message: PCB Save: 1 files changed mainbrd3.kicad_pcb 257/0/873
Parts:
- C16: moved to B.Cu
- moved J4 153.2 mm to (199.8, 99.6)
- moved D6 145.0 mm to (157.4, 116.1), turned to 90 degrees
- moved D5 144.4 mm to (155.6, 116.1), turned to 90 degrees
- moved R42 125.7 mm to (157.1, 113.0), turned to 90 degrees
- moved R41 125.7 mm to (155.9, 113.0), turned to 90 degrees
- moved J10 112.7 mm to (141.4, 108.9)
- moved R3 104.6 mm to (132.2, 101.8)
- moved R4 104.6 mm to (132.2, 103.8)
- moved J3 102.3 mm to (138.6, 100.0), turned to 180 degrees
- moved J1 89.7 mm to (135.8, 84.2), turned to 90 degrees
- moved C16 34.7 mm to (121.7, 81.2), turned to -90 degrees
- moved C33 34.4 mm to (132.7, 76.4), turned to -90 degrees
- moved C17 0.10 mm to (164.9, 104.5)
Routing:
- net Net-(U1-PF5): track 0.00 -> 10.9 mm
- net Net-(U1-PF4): track 0.00 -> 10.6 mm
- net GND: track 85.6 -> 92.9 mm, vias 66 -> 68
- net Net-(U2-SS): track 0.00 -> 3.06 mm, vias 0 -> 1
- net Net-(D6-A): track 0.00 -> 1.92 mm
- net Net-(D5-A): track 0.00 -> 1.90 mm
- net /MCU/3v3_usb: track 0.00 -> 0.70 mm
- added copper zone on F.Cu, net +3V3VADC
- removed copper zone on B.Cu, net +3V3VADC

Commit message: PCB Save: 2 files changed mainbrd3.kicad_pcb 679/0/2551 mainbrd3.kicad_prl 0/0/1
Parts:
- moved R4 67.0 mm to (199.2, 105.5)
- moved J10 45.3 mm to (168.4, 72.5), turned to 180 degrees
- moved R3 12.7 mm to (140.7, 92.4), turned to 180 degrees
- moved R25 6.35 mm to (155.1, 74.8)
- moved R27 6.35 mm to (155.1, 76.0)
- moved R28 6.35 mm to (159.6, 69.3)
- moved U5 6.35 mm to (160.2, 74.1)
- moved R26 6.35 mm to (155.1, 73.5)
- moved J3 3.30 mm to (141.2, 98.0)
- moved J1 2.00 mm to (133.8, 84.7)
Routing:
- net SWDIO: track 0.00 -> 17.6 mm
- net BOOT0: track 0.00 -> 17.3 mm, vias 0 -> 1
- net NRST: track 49.1 -> 60.3 mm
- net SWCLK: track 0.00 -> 10.4 mm
- net I2C1_SDA: track 43.0 -> 35.8 mm
- net I2C1_SCL: track 41.8 -> 34.7 mm
- net GND: track 92.9 -> 98.2 mm, vias 68 -> 70
- net +3V3: track 58.6 -> 63.6 mm, vias 39 -> 41
- net Earth: track 38.5 -> 39.3 mm
- net D+: track 16.7 -> 17.2 mm
- net D-: track 16.7 -> 17.2 mm
- net Net-(U5-A0): track 3.02 -> 2.90 mm, vias 1 -> 0
