File: REVA1-2.kicad_pcb (KiCad board)
At the start: 4 copper layers, 100 x 72 mm, 110 parts, among them J1 Conn_01x04_Pin, J10 Conn_01x03_Pin, J2 USB_B_Micro, J3 Conn_01x02_Pin, J4 Conn_01x02_Pin, J5 https://abracon.com/Magnetics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, J6 Screw_Terminal_01x02, J7 Screw_Terminal_01x02, J8 Screw_Terminal_01x02, J9 Screw_Terminal_01x02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

Commit message: Autosave
Parts:
- moved R5 0.93 mm to (188.5, 81.9), turned to 90 degrees
- moved C30 0.40 mm to (185.7, 81.8)
Routing:
- net Earth: track 47.0 -> 39.3 mm
- net GND: track 104.6 -> 102.2 mm, vias 70 -> 69
- net +5VUSB: track 4.59 -> 2.22 mm
- net /ETH/Erx+: track 27.2 -> 25.6 mm
- net /ETH/Etx+: track 26.0 -> 24.5 mm
- net +3V3_ethtxrx: track 67.2 -> 65.8 mm
- net Net-(U3-RBIAS): track 7.36 -> 6.22 mm
- net Net-(C31-Pad1): track 10.5 -> 9.48 mm
- net /ETH/Erx-: track 27.6 -> 26.9 mm
- net UART4_RX: vias 2 -> 3
