File: untitled.kicad_sch (KiCad schematic)
At the start: 60 parts, among them J1 Conn_01x04_Pin, J10 Conn_01x03_Pin, J2 USB_B_Micro, J3 Conn_01x02_Pin, J4 Conn_01x02_Pin, J6 Screw_Terminal_01x02, J9 Screw_Terminal_01x02, U1 STM32F767ZITx, U2 MAX17501AATB+, U5 AT24C256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

Commit message: SCH Save: 1 files changed untitled.kicad_sch 0/10/205
Connections:
- net D+: now also U1.104 (PA12); no longer U1.76 (PB15)
- net D-: now also U1.103 (PA11); no longer U1.75 (PB14)
- net UART4_DIR: now also U1.110 (PA15); no longer U1.102 (PA10)
- net UART4_RX: now also U1.112 (PC11); no longer U1.103 (PA11)
- net UART4_TX: now also U1.111 (PC10); no longer U1.104 (PA12)
- net UART5_DIR: now also U1.98 (PC8); no longer U1.117 (PD3)
- net UART3_TX: now reaches U1.77 (PD8)
- net UART3_TX: now also J10.1 (Pin_1)
- net UART3_RX: now reaches U1.78 (PD9)
- net UART3_RX: now also J10.2 (Pin_2)
- net UART8_RX: no longer names the net of U1.141 (PE0)
- net UART8_RX: no longer J10.1 (Pin_1)
- net UART8_TX: no longer names the net of U1.142 (PE1)
- net UART8_TX: no longer J10.2 (Pin_2)
- no-connect marks 96 -> 93
Other:
- moved on the sheet: J10

Commit message: SCH Save: 1 files changed untitled.kicad_sch 0/617/2
Parts:
- removed D2: MBR0580, Diode_SMD:D_SOD-123, symbol Diode:MBR0580
- removed F2: Fuse, Fuse:Fuse_1206_3216Metric, symbol Device:Fuse

Commit message: Autosave
Parts:
- J2, U2: now fitted
Connections:
- net Earth: now also J2.6 (Shield)
- no-connect marks 93 -> 92
Changed lines of the file:
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@@
 	)
 	(no_connect
-		(at 382.27 52.07)
-	)
-	(no_connect
 		(at 111.76 182.88)
 	)
@@
 	(wire
 		(pts
+			(xy 382.27 45.72) (xy 384.81 45.72)
+		)
+		(stroke
+			(width 0)
+			(type default)
+		)
+	)
+	(wire
+		(pts
 			(xy 166.37 41.91) (xy 177.8 41.91)
 		)
@@
 	(wire
 		(pts
+			(xy 382.27 45.72) (xy 382.27 52.07)
+		)
+		(stroke
+			(width 0)
+			(type default)
+		)
+	)
+	(wire
+		(pts
 			(xy 172.72 200.66) (xy 189.23 200.66)
 		)
@@
 		)
 	)
+	(global_label "Earth"
+		(shape input)
+		(at 384.81 45.72 0)
+		(fields_autoplaced yes)
+		(effects
+			(font
+				(size 1.27 1.27)
+			)
+			(justify left)
+		)
+		(property "Intersheetrefs" "${INTERSHEET_REFS}"
+			(at 392.7541 45.72 0)
+			(hide yes)
+			(show_name no)
+			(do_not_autoplace no)
+			(effects
+				(font
+					(size 1.27 1.27)
+				)
+				(justify left)
+			)
+		)
+	)
 	(global_label "I2C1_SCL"
 		(shape input)
@@
 		(on_board yes)
 		(in_pos_files yes)
-		(dnp yes)
+		(dnp no)
 		(fields_autoplaced yes)
 		(property "Reference" "U2"
@@
 		(on_board yes)
 		(in_pos_files yes)
-		(dnp yes)
+		(dnp no)
 		(fields_autoplaced yes)
 		(property "Reference" "J2"

Commit message: asf
Connections:
- net Earth: now also J2.SH (Shield); no longer J2.6 (Shield)
Changed lines of the file:
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@@
 		(pin "1"
 		)
-		(pin "6"
+		(pin "SH"
 		)
 		(pin "2"

Commit message: Autosave
Connections:
- net Earth: now also J2.6 (Shield); no longer J2.SH (Shield)
Changed lines of the file:
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@@
 		(pin "1"
 		)
-		(pin "SH"
+		(pin "6"
 		)
 		(pin "2"

Commit message: Autosave
Parts:
- C1, C2: MPN (none) -> 0402CG100J500NT
- C10, C11, C12, C3, C34, C4, C5, C6, C7, C8, C9: MPN (none) -> 0402F104M500NT
- C13: MPN (none) -> CL10A106MQ8NNNC
- C14: MPN (none) -> CL31B105KCHNNNE
- C15, C17, C32, C33: MPN (none) -> CL05A105KP5NNNC
- C16: MPN (none) -> 0402B332K500NT
- C18: MPN (none) -> 0402B103K500NT
- C19: MPN (none) -> CC0603KRX5R8BB105
- C20: JLCPCB PN C1691 -> C1691; MPN (none) -> CL10A106MQ8NNNC
- D1: MPN (none) -> MBR0580
- D5, D6: MPN (none) -> KT-0603R
- F1: MPN (none) -> SMD1206P016TF
- L1: MPN (none) -> FNR4018S270MT
- L3: MPN (none) -> MCL2012S1R0MT
- R1: MPN (none) -> CR0402JF0335G
- R2: MPN (none) -> RC-02W300JT
- R23, R24: MPN (none) -> 0402WGF2001TCE
- R25, R26, R27, R28: MPN (none) -> 0402WGF2000TCE
- R3, R4: MPN (none) -> 0402WGJ0103TCE
- R41, R42: MPN (none) -> 0402WGJ0361TCE
- U1: MPN (none) -> STM32F767ZIT6
- U5: MPN (none) -> AT24C256C-SSHL-T
- U8: MPN (none) -> AMS1117-3.3
- Y1: MPN (none) -> WTL3M01610

Commit message: Autosave
Parts:
- added PS1: RI3-1205S, joefplib:CONV_RI3-1205S, symbol joelib:RI3-1205S
Changed lines of the file:
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@@
+	)
+	(symbol
+		(lib_id "joelib:RI3-1205S")
+		(at 231.14 160.02 0)
+		(unit 1)
+		(body_style 1)
+		(exclude_from_sim no)
+		(in_bom yes)
+		(on_board yes)
+		(in_pos_files yes)
+		(dnp no)
+		(fields_autoplaced yes)
+		(property "Reference" "PS1"
+			(at 231.14 147.32 0)
+			(show_name no)
+			(do_not_autoplace no)
+			(effects
+				(font
+					(size 1.27 1.27)
+				)
+			)
+		)
+		(property "Value" "RI3-1205S"
+			(at 231.14 149.86 0)
+			(show_name no)
+			(do_not_autoplace no)
+			(effects
+				(font
+					(size 1.27 1.27)
+				)
+			)
+		)
+		(property "Footprint" "joefplib:CONV_RI3-1205S"
+			(at 231.14 160.02 0)
+			(hide yes)
+			(show_name no)
+			(do_not_autoplace no)
+			(effects
+				(font
+					(size 1.27 1.27)
+				)
+				(justify bottom)
+			)
+		)
+		(property "Datasheet" ""
+			(at 231.14 160.02 0)
+			(hide yes)
+			(show_name no)
+			(do_not_autoplace no)
+			(effects
+				(font
+					(size 1.27 1.27)
+				)
+			)
+		)
+		(property "Description" ""
+			(at 231.14 160.02 0)
+			(hide yes)
+			(show_name no)
+			(do_not_autoplace no)
+			(effects
+				(font
+					(size 1.27 1.27)
+				)
+			)
+		)
+		(property "PARTREV" "3"
+			(at 231.14 160.02 0)
+			(hide yes)
+			(show_name no)
+			(do_not_autoplace no)
+			(effects
+				(font
+					(size 1.27 1.27)
+				)
+				(justify bottom)
+			)
+		)
+		(property "STANDARD" "Manufacturer Recommendations"
+			(at 231.14 160.02 0)
+			(hide yes)
+			(show_name no)
+			(do_not_autoplace no)
+			(effects
+				(font
+					(size 1.27 1.27)
+				)
+				(justify bottom)
+			)
+		)
+		(property "MAXIMUM_PACKAGE_HEIGHT" "10.2mm"
+			(at 231.14 160.02 0)
+			(hide yes)
+			(show_name no)
+			(do_not_autoplace no)
+			(effects
+				(font
+					(size 1.27 1.27)
+				)
+				(justify bottom)
+			)
+		)
+		(property "MANUFACTURER" "Recom"
+			(at 231.14 160.02 0)
+			(hide yes)
+			(show_name no)
+			(do_not_autoplace no)
+			(effects
+				(font
+					(size 1.27 1.27)
+				)
+				(justify bottom)
+			)
+		)
+		(pin "2"
+		)
+		(pin "4"
+		)
+		(pin "3"
+		)
+		(pin "1"
+		)
+		(instances
+			(project "mainbrd3"
+				(path "/89e0f049-91ab-4c37-b514-d5ee0e775d39/5a91110a-5d39-48c9-af7e-bae13d852cb2"
+					(reference "PS1")
+					(unit 1)
+				)
+			)
+		)
 	)
 	(symbol

Commit message: Autosave
Parts:
- removed C14: 1uF, Capacitor_SMD:C_1206_3216Metric, symbol Device:C
- removed C16: 3300pF, Capacitor_SMD:C_0402_1005Metric, symbol Device:C
- removed C19: 1uF, Capacitor_SMD:C_0603_1608Metric, symbol Device:C
- removed C20: 10uF, Capacitor_SMD:C_0603_1608Metric, symbol Device:C
- removed D1: MBR0580, Diode_SMD:D_SOD-123, symbol Diode:MBR0580
- removed F1: Fuse, Fuse:Fuse_1206_3216Metric, symbol Device:Fuse
- removed L1: 26.6uH, Inductor_SMD:L_Changjiang_FNR4018S, symbol Device:L
- removed R1: 3300k, Resistor_SMD:R_0402_1005Metric, symbol Device:R
- removed R2: 600k, Resistor_SMD:R_0402_1005Metric, symbol Device:R
- removed U2: MAX17501AATB+, Package_DFN_QFN:TDFN-10-1EP_2x3mm_P0.5mm_EP0.9x2mm, symbol Regulator_Switching:MAX17501AxTB
Connections:
- net 3v3smps is gone; now on an unnamed net: JP1.3 (B)
- net GND: now also PS1.3 (-VOUT)
- no-connect marks 92 -> 91
Other:
- note removed: "X7R 1206"
- note removed: "X7R min 1μF min 80v In applications where the source is located distant from the device input, an electrolytic capacitor should be added in parallel to the 1μF ceramic capacitor to provide necessary damping for potential oscillations caused by the longer input power path and input ceramic capacitor."
- moved on the sheet: PS1
