File: untitled.kicad_sch (KiCad schematic)
At the start: 49 parts, among them J1 Conn_01x04_Pin, J10 Conn_01x03_Pin, J2 USB_B_Micro, J3 Conn_01x02_Pin, J4 Conn_01x02_Pin, J6 Screw_Terminal_01x02, J9 Screw_Terminal_01x02, U1 STM32F767ZITx, U5 AT24C256, U8 AMS1117-3.3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

Commit message: Autosave
Parts:
- added U9: AMS1117-3.3, Package_TO_SOT_SMD:SOT-223-3_TabPin2, symbol Regulator_Linear:AMS1117-3.3
Connections:
- net +12V: now also PS1.2 (+VIN)
- net GND: now also U9.1 (GND); no longer J9.2 (Pin_2)
- net at JP1.3 (B): now also U9.2 (VO); no longer PS1.4 (+VOUT)
- net GND1: now reaches PS1.1 (-VIN)
- net GND1: now also J9.2 (Pin_2)
- new net: PS1.4 (+VOUT), U9.3 (VI)
Other:
- moved on the sheet: PS1

Commit message: Autosave
Connections:
- net +3.3V_dcdc: now reaches JP1.3 (B), U9.2 (VO)
- no-connect marks 91 -> 92

Commit message: Autosave
Connections:
- no-connect marks 92 -> 94

Commit message: Autosave
Changed lines of the file:
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@@
 	)
 	(junction
-		(at 361.95 111.76)
-		(diameter 0)
-		(color 0 0 0 0)
-	)
-	(junction
 		(at 76.2 34.29)
 		(diameter 0)
@@
 	(wire
 		(pts
+			(xy 359.41 111.76) (xy 369.57 111.76)
+		)
+		(stroke
+			(width 0)
+			(type default)
+		)
+	)
+	(wire
+		(pts
 			(xy 119.38 34.29) (xy 130.81 34.29)
 		)
@@
 	(wire
 		(pts
-			(xy 359.41 111.76) (xy 361.95 111.76)
-		)
-		(stroke
-			(width 0)
-			(type default)
-		)
-	)
-	(wire
-		(pts
 			(xy 368.3 85.09) (xy 368.3 86.36)
 		)
@@
 	(wire
 		(pts
-			(xy 361.95 111.76) (xy 369.57 111.76)
-		)
-		(stroke
-			(width 0)
-			(type default)
-		)
-	)
-	(wire
-		(pts
 			(xy 382.27 85.09) (xy 392.43 85.09)
 		)
@@
 					(unit 1)
 				)
-			)
-		)
-	)
-	(symbol
-		(lib_id "power:PWR_FLAG")
-		(at 361.95 111.76 0)
-		(unit 1)
-		(body_style 1)
-		(exclude_from_sim no)
-		(in_bom yes)
-		(on_board yes)
-		(in_pos_files yes)
-		(dnp no)
-		(fields_autoplaced yes)
-		(property "Reference" "#FLG011"
-			(at 361.95 109.855 0)
-			(hide yes)
-			(show_name no)
-			(do_not_autoplace no)
-			(effects
-				(font
-					(size 1.27 1.27)
-				)
-			)
-		)
-		(property "Value" "PWR_FLAG"
-			(at 361.95 106.68 0)
-			(show_name no)
-			(do_not_autoplace no)
-			(effects
-				(font
-					(size 1.27 1.27)
-				)
-			)
-		)
-		(property "Footprint" ""
-			(at 361.95 111.76 0)
-			(hide yes)
-			(show_name no)
-			(do_not_autoplace no)
-			(effects
-				(font
-					(size 1.27 1.27)
-				)
-			)
-		)
-		(property "Datasheet" ""
-			(at 361.95 111.76 0)
-			(hide yes)
-			(show_name no)
-			(do_not_autoplace no)
-			(effects
-				(font
-					(size 1.27 1.27)
-				)
-			)
-		)
-		(property "Description" "Special symbol for telling ERC where power comes from"
-			(at 361.95 111.76 0)
-			(hide yes)
-			(show_name no)
-			(do_not_autoplace no)
-			(effects
-				(font
-					(size 1.27 1.27)
-				)
-			)
-		)
-		(pin "1"
-		)
-		(instances
-			(project "mainbrd3"
-				(path "/89e0f049-91ab-4c37-b514-d5ee0e775d39/5a91110a-5d39-48c9-af7e-bae13d852cb2"
-					(reference "#FLG011")
-					(unit 1)
-				)

Commit message: Autosave
Parts:
- added C14: 10uf, Capacitor_SMD:C_0805_2012Metric, symbol Device:C
- added C16, C20, C35: 10uf, Capacitor_Tantalum_SMD:CP_EIA-3216-18_Kemet-A, symbol Device:C_Polarized
- added C19, C36: 100nf, Capacitor_SMD:C_0402_1005Metric, symbol Device:C
- added F1: Fuse, Fuse:Fuse_0603_1608Metric_Pad1.05x0.95mm_HandSolder, symbol Device:Fuse
Connections:
- net +12V: now also F1.1; no longer PS1.2 (+VIN)
- net +3.3V_dcdc: now also C20.1, C35.1, C36.1
- net GND: now also C16.2, C19.2, C20.2, C35.2, C36.2
- net GND1: now also C14.2
- net at PS1.4 (+VOUT), U9.3 (VI): now also C16.1, C19.1
- new net: C14.1, F1.2, PS1.2 (+VIN)
Other:
- moved on the sheet: PS1, U9
