File: untitled.kicad_sch (KiCad schematic)
At the start: 57 parts, among them J1 Conn_01x04_Pin, J10 Conn_01x03_Pin, J2 USB_B_Micro, J3 Conn_01x02_Pin, J4 Conn_01x02_Pin, J6 Screw_Terminal_01x02, J9 Screw_Terminal_01x02, U1 STM32F767ZITx, U5 AT24C256, U8 AMS1117-3.3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

Commit message: Autosave
Parts:
- C14: value 10uf -> 47uf; footprint Capacitor_SMD:C_0805_2012Metric -> Capacitor_SMD:C_1210_3225Metric; LCSC C440198 -> C77101; MPN GRM21BR61H106KE43L -> GRM32ER61C476KE15L
Changed lines of the file:
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@@
 			)
 		)
-		(property "Value" "10uf"
+		(property "Value" "47uf"
 			(at 298.45 118.1099 0)
 			(show_name no)
@@
 			)
 		)
-		(property "Footprint" "Capacitor_SMD:C_0805_2012Metric"
+		(property "Footprint" "Capacitor_SMD:C_1210_3225Metric"
 			(at 295.6052 120.65 0)
 			(hide yes)
@@
 			)
 		)
-		(property "MPN" "GRM21BR61H106KE43L"
+		(property "MPN" " GRM32ER61C476KE15L"
 			(at 294.64 116.84 0)
 			(hide yes)
@@
 			)
 		)
-		(property "LCSC" "C440198"
+		(property "LCSC" " C77101"
 			(at 294.64 116.84 0)
 			(hide yes)
@@
 		)
 	)
-	(group ""
-		(members "535b15c4-0c5b-4b06-bde4-9105bbb0638f")
-	)
 )

Commit message: Autosave
Connections:
- net +12V: now also C14.1, F1.2, PS1.2 (+VIN); no longer F1.1, J9.1 (Pin_1)
- new net +12VIN: F1.1, J9.1 (Pin_1)
Changed lines of the file:
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@@
 	)
 	(junction
+		(at 288.29 111.76)
+		(diameter 0)
+		(color 0 0 0 0)
+	)
+	(junction
 		(at 279.4 241.3)
 		(diameter 0)
@@
 	(wire
 		(pts
+			(xy 288.29 111.76) (xy 294.64 111.76)
+		)
+		(stroke
+			(width 0)
+			(type default)
+		)
+	)
+	(wire
+		(pts
 			(xy 71.12 55.88) (xy 127 55.88)
 		)
@@
 	(wire
 		(pts
-			(xy 283.21 111.76) (xy 294.64 111.76)
+			(xy 283.21 111.76) (xy 288.29 111.76)
 		)
 		(stroke
@@
 			)
 		)
-		(property "Value" "+12V"
+		(property "Value" "+12VIN"
 			(at 293.37 20.32 0)
 			(show_name no)
@@
 			)
 		)
-		(property "Value" "+12V"
+		(property "Value" "+12VIN"
 			(at 283.21 87.63 0)
 			(show_name no)
@@
 					(unit 1)
 				)
+			)
+		)
+	)
+	(symbol
+		(lib_id "power:+12V")
+		(at 288.29 111.76 0)
+		(unit 1)
+		(body_style 1)
+		(exclude_from_sim no)
+		(in_bom yes)
+		(on_board yes)
+		(in_pos_files yes)
+		(dnp no)
+		(fields_autoplaced yes)
+		(property "Reference" "#PWR012"
+			(at 288.29 115.57 0)
+			(hide yes)
+			(show_name no)
+			(do_not_autoplace no)
+			(effects
+				(font
+					(size 1.27 1.27)
+				)
+			)
+		)
+		(property "Value" "+12V"
+			(at 288.29 106.68 0)
+			(show_name no)
+			(do_not_autoplace no)
+			(effects
+				(font
+					(size 1.27 1.27)
+				)
+			)
+		)
+		(property "Footprint" ""
+			(at 288.29 111.76 0)
+			(hide yes)
+			(show_name no)
+			(do_not_autoplace no)
+			(effects
+				(font
+					(size 1.27 1.27)
+				)
+			)
+		)
+		(property "Datasheet" ""
+			(at 288.29 111.76 0)
+			(hide yes)
+			(show_name no)
+			(do_not_autoplace no)
+			(effects
+				(font
+					(size 1.27 1.27)
+				)
+			)
+		)
+		(property "Description" "Power symbol creates a global label with name \"+12V\""
+			(at 288.29 111.76 0)
+			(hide yes)
+			(show_name no)
+			(do_not_autoplace no)
+			(effects
+				(font
+					(size 1.27 1.27)
+				)
+			)
+		)
+		(pin "1"
+		)
+		(instances
+			(project "mainbrd3"
+				(path "/89e0f049-91ab-4c37-b514-d5ee0e775d39/5a91110a-5d39-48c9-af7e-bae13d852cb2"
+					(reference "#PWR012")
+					(unit 1)
+				)

Commit message: Autosave
Parts:
- removed J6: Screw_Terminal_01x02, TerminalBlock_Phoenix:TerminalBlock_Phoenix_MKDS-1,5-2-5.08_1x02_P5.08mm_Horizontal, symbol Connector:Screw_Terminal_01x02
Connections:
- no-connect marks 94 -> 93
Changed lines of the file:
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@@
 	)
 	(no_connect
-		(at 252.73 26.67)
-	)
-	(no_connect
 		(at 172.72 198.12)
 	)
@@
 	(wire
 		(pts
-			(xy 251.46 24.13) (xy 252.73 24.13)
-		)
-		(stroke
-			(width 0)
-			(type default)
-		)
-	)
-	(wire
-		(pts
 			(xy 369.57 120.65) (xy 369.57 121.92)
 		)
@@
 	(wire
 		(pts
-			(xy 251.46 24.13) (xy 251.46 30.48)
-		)
-		(stroke
-			(width 0)
-			(type default)
-		)
-	)
-	(wire
-		(pts
 			(xy 293.37 26.67) (xy 293.37 24.13)
 		)
@@
 	(wire
 		(pts
-			(xy 248.92 30.48) (xy 251.46 30.48)
-		)
-		(stroke
-			(width 0)
-			(type default)
-		)
-	)
-	(wire
-		(pts
 			(xy 81.28 143.51) (xy 81.28 147.32)
 		)
@@
 	)
 	(symbol
-		(lib_id "Connector:Screw_Terminal_01x02")
-		(at 257.81 24.13 0)
-		(unit 1)
-		(body_style 1)
-		(exclude_from_sim no)
-		(in_bom yes)
-		(on_board yes)
-		(in_pos_files yes)
-		(dnp yes)
-		(fields_autoplaced yes)
-		(property "Reference" "J6"
-			(at 260.35 24.1299 0)
-			(show_name no)
-			(do_not_autoplace no)
-			(effects
-				(font
-					(size 1.27 1.27)
-				)
-				(justify left)
-			)
-		)
-		(property "Value" "Screw_Terminal_01x02"
-			(at 260.35 26.6699 0)
-			(show_name no)
-			(do_not_autoplace no)
-			(effects
-				(font
-					(size 1.27 1.27)
-				)
-				(justify left)
-			)
-		)
-		(property "Footprint" "TerminalBlock_Phoenix:TerminalBlock_Phoenix_MKDS-1,5-2-5.08_1x02_P5.08mm_Horizontal"
-			(at 257.81 24.13 0)
-			(hide yes)
-			(show_name no)
-			(do_not_autoplace no)
-			(effects
-				(font
-					(size 1.27 1.27)
-				)
-			)
-		)
-		(property "Datasheet" ""
-			(at 257.81 24.13 0)
-			(hide yes)
-			(show_name no)
-			(do_not_autoplace no)
-			(effects
-				(font
-					(size 1.27 1.27)
-				)
-			)
-		)
-		(property "Description" "Generic screw terminal, single row, 01x02, script generated (kicad-library-utils/schlib/autogen/connector/)"
-			(at 257.81 24.13 0)
-			(hide yes)
-			(show_name no)
-			(do_not_autoplace no)
-			(effects
-				(font
-					(size 1.27 1.27)
-				)
-			)
-		)
-		(property "MPN" ""
-			(at 257.81 24.13 0)
-			(hide yes)
-			(show_name no)
-			(do_not_autoplace no)
-			(effects
-				(font
-					(size 1.27 1.27)
-				)
-			)
-		)
-		(pin "1"
-		)
-		(pin "2"
-		)
-		(instances
-			(project "mainbrd3"
-				(path "/89e0f049-91ab-4c37-b514-d5ee0e775d39/5a91110a-5d39-48c9-af7e-bae13d852cb2"
-					(reference "J6")
-					(unit 1)
-				)
-			)
-		)
-	)
-	(symbol
 		(lib_id "Device:C_Polarized")
 		(at 378.46 116.84 0)
@@
 					(unit 1)
 				)
-			)
-		)
-	)
-	(symbol
-		(lib_id "power:Earth")
-		(at 248.92 30.48 0)
-		(unit 1)
-		(body_style 1)
-		(exclude_from_sim no)
-		(in_bom yes)
-		(on_board yes)
-		(in_pos_files yes)
-		(dnp no)
-		(fields_autoplaced yes)
-		(property "Reference" "#PWR057"
-			(at 248.92 36.83 0)
-			(hide yes)
-			(show_name no)
-			(do_not_autoplace no)
-			(effects
-				(font
-					(size 1.27 1.27)
-				)
-			)
-		)
-		(property "Value" "Earth"
-			(at 248.92 35.56 0)
-			(show_name no)
-			(do_not_autoplace no)
-			(effects
-				(font
-					(size 1.27 1.27)
-				)
-			)
-		)
-		(property "Footprint" ""
-			(at 248.92 30.48 0)
-			(hide yes)
-			(show_name no)
-			(do_not_autoplace no)
-			(effects
-				(font
-					(size 1.27 1.27)
-				)
-			)
-		)
-		(property "Datasheet" ""
-			(at 248.92 30.48 0)
-			(hide yes)
-			(show_name no)
-			(do_not_autoplace no)
-			(effects
-				(font
-					(size 1.27 1.27)
-				)
-			)
-		)
-		(property "Description" "Power symbol creates a global label with name \"Earth\""
-			(at 248.92 30.48 0)
-			(hide yes)
-			(show_name no)
-			(do_not_autoplace no)
-			(effects
-				(font
-					(size 1.27 1.27)
-				)
-			)
-		)
-		(pin "1"
-		)
-		(instances
-			(project "mainbrd3"
-				(path "/89e0f049-91ab-4c37-b514-d5ee0e775d39/5a91110a-5d39-48c9-af7e-bae13d852cb2"
-					(reference "#PWR057")
-					(unit 1)
-				)

Commit message: Autosave
Connections:
- net Relay_signal: now reaches U1.114 (PD0)
- no-connect marks 93 -> 92
Changed lines of the file:
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@@
 	)
 	(no_connect
-		(at 172.72 195.58)
-	)
-	(no_connect
 		(at 172.72 175.26)
 	)
@@
 	(wire
 		(pts
+			(xy 172.72 195.58) (xy 189.23 195.58)
+		)
+		(stroke
+			(width 0)
+			(type default)
+		)
+	)
+	(wire
+		(pts
 			(xy 254 60.96) (xy 254 58.42)
 		)
@@
 		)
 	)
+	(label "Relay_Signal"
+		(at 176.53 195.58 0)
+		(effects
+			(font
+				(size 1.27 1.27)
+			)
+			(justify left bottom)
+		)
+	)
 	(label "3v3_usb"
 		(at 368.3 85.09 0)
@@
 			(hide yes)
 			(show_name no)
+			(do_not_autoplace no)
+			(effects
+				(font
+					(size 1.27 1.27)
+				)
+				(justify left)
+			)
+		)
+	)
+	(global_label "Relay_signal"
+		(shape input)
+		(at 189.23 195.58 0)
+		(fields_autoplaced yes)
+		(effects
+			(font
+				(size 1.27 1.27)
+			)
+			(justify left)
+		)
+		(property "Intersheetrefs" "${INTERSHEET_REFS}"
+			(at 204.0683 195.58 0)
+			(hide yes)
+			(show_name no)
