File: sheet3.kicad_sch (KiCad schematic)
At the start: 18 parts, among them J7 Screw_Terminal_01x02, J8 Screw_Terminal_01x02, U6 MAX3485, U7 MAX3485

Commit message: SCH Save: 1 files changed sheet3.kicad_sch 0/2/12
Connections:
- net at D3.2 (A2), R33.2, R34.1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: now also J7.1 (Pin_1); no longer J7.2 (Pin_2)
- net at D3.1 (A1), R32.1, R34.2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: now also J7.2 (Pin_2); no longer J7.1 (Pin_1)
- net at D4.2 (A2), R38.2, R40.1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: now also J8.1 (Pin_1); no longer J8.2 (Pin_2)
- net at D4.1 (A1), R39.1, R40.2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: now also J8.2 (Pin_2); no longer J8.1 (Pin_1)
Changed lines of the file:
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@@
 	(symbol
 		(lib_id "Connector:Screw_Terminal_01x02")
-		(at 163.83 45.72 0)
-		(mirror x)
+		(at 163.83 43.18 0)
 		(unit 1)
 		(body_style 1)
@@
 		(dnp yes)
 		(property "Reference" "J7"
-			(at 166.37 45.7201 0)
+			(at 166.37 43.1799 0)
 			(show_name no)
 			(do_not_autoplace no)
@@
 		)
 		(property "Value" "Screw_Terminal_01x02"
-			(at 166.37 43.1801 0)
+			(at 166.37 45.7199 0)
 			(show_name no)
 			(do_not_autoplace no)
@@
 		)
 		(property "Footprint" "TerminalBlock_Phoenix:TerminalBlock_Phoenix_MKDS-1,5-2-5.08_1x02_P5.08mm_Horizontal"
-			(at 163.83 45.72 0)
+			(at 163.83 43.18 0)
 			(hide yes)
 			(show_name no)
@@
 		)
 		(property "Datasheet" ""
-			(at 163.83 45.72 0)
+			(at 163.83 43.18 0)
 			(hide yes)
 			(show_name no)
@@
 		)
 		(property "Description" "Generic screw terminal, single row, 01x02, script generated (kicad-library-utils/schlib/autogen/connector/)"
-			(at 163.83 45.72 0)
+			(at 163.83 43.18 0)
 			(hide yes)
 			(show_name no)
@@
 	(symbol
 		(lib_id "Connector:Screw_Terminal_01x02")
-		(at 163.83 99.06 0)
-		(mirror x)
+		(at 163.83 96.52 0)
 		(unit 1)
 		(body_style 1)
@@
 		(dnp yes)
 		(property "Reference" "J8"
-			(at 166.37 99.0601 0)
+			(at 166.37 96.5199 0)
 			(show_name no)
 			(do_not_autoplace no)
@@
 		)
 		(property "Value" "Screw_Terminal_01x02"
-			(at 166.37 96.5201 0)
+			(at 166.37 99.0599 0)
 			(show_name no)
 			(do_not_autoplace no)
@@
 		)
 		(property "Footprint" "TerminalBlock_Phoenix:TerminalBlock_Phoenix_MKDS-1,5-2-5.08_1x02_P5.08mm_Horizontal"
-			(at 163.83 99.06 0)
+			(at 163.83 96.52 0)
 			(hide yes)
 			(show_name no)
@@
 		)
 		(property "Datasheet" ""
-			(at 163.83 99.06 0)
+			(at 163.83 96.52 0)
 			(hide yes)
 			(show_name no)
@@
 		)
 		(property "Description" "Generic screw terminal, single row, 01x02, script generated (kicad-library-utils/schlib/autogen/connector/)"
-			(at 163.83 99.06 0)
-			(hide yes)
-			(show_name no)
+			(at 163.83 96.52 0)
+			(hide yes)
+			(show_name no)

Commit message: Autosave
Parts:
- D3, D4: MPN (none) -> SM712
- R29, R30, R31, R32, R33, R35, R36, R37, R38, R39: MPN (none) -> 0402WGJ0103TCE
- R34, R40: MPN (none) -> 0402WGF1200TCE
- U6, U7: MPN (none) -> MAX3485ESA(UMW)
Changed lines of the file:
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@@
+			)
+		)
+		(property "MPN" "0402WGJ0103TCE"
+			(at 49.53 34.29 0)
+			(hide yes)
+			(show_name no)
+			(do_not_autoplace no)
+			(effects
+				(font
+					(size 1.27 1.27)
+				)
 			)
 		)
@@
 			)
 		)
+		(property "MPN" "MAX3485ESA(UMW)"
+			(at 80.01 49.53 0)
+			(hide yes)
+			(show_name no)
+			(do_not_autoplace no)
+			(effects
+				(font
+					(size 1.27 1.27)
+				)
+			)
+		)
 		(pin "2"
 		)
@@
 			)
 		)
+		(property "MPN" ""
+			(at 163.83 43.18 0)
+			(hide yes)
+			(show_name no)
+			(do_not_autoplace no)
+			(effects
+				(font
+					(size 1.27 1.27)
+				)
+			)
+		)
 		(pin "1"
 		)
@@
 			)
 		)
+		(property "MPN" "0402WGF1200TCE"
+			(at 137.16 97.79 0)
+			(hide yes)
+			(show_name no)
+			(do_not_autoplace no)
+			(effects
+				(font
+					(size 1.27 1.27)
+				)
+			)
+		)
 		(pin "2"
 		)
@@
 			)
 		)
+		(property "MPN" "0402WGJ0103TCE"
+			(at 96.52 106.68 0)
+			(hide yes)
+			(show_name no)
+			(do_not_autoplace no)
+			(effects
+				(font
+					(size 1.27 1.27)
+				)
+			)
+		)
 		(pin "2"
 		)
@@
 			)
 		)
+		(property "MPN" "0402WGJ0103TCE"
+			(at 57.15 34.29 0)
+			(hide yes)
+			(show_name no)
+			(do_not_autoplace no)
+			(effects
+				(font
+					(size 1.27 1.27)
+				)
+			)
+		)
 		(pin "2"
 		)
@@
 			)
 		)
+		(property "MPN" "0402WGJ0103TCE"
+			(at 49.53 87.63 0)
+			(hide yes)
+			(show_name no)
+			(do_not_autoplace no)
+			(effects
+				(font
+					(size 1.27 1.27)
+				)
+			)
+		)
 		(pin "2"
 		)
@@
 			)
 		)
+		(property "MPN" "0402WGJ0103TCE"
+			(at 96.52 34.29 0)
+			(hide yes)
+			(show_name no)
+			(do_not_autoplace no)
+			(effects
+				(font
+					(size 1.27 1.27)
+				)
+			)
+		)
 		(pin "2"
 		)
@@
 			)
 		)
+		(property "MPN" "SM712"
+			(at 121.92 97.79 90)
+			(hide yes)
+			(show_name no)
+			(do_not_autoplace no)
+			(effects
+				(font
+					(size 1.27 1.27)
+				)
+			)
+		)
 		(pin "1"
 		)
@@
 			)
 		)
+		(property "MPN" "0402WGJ0103TCE"
+			(at 96.52 53.34 0)
+			(hide yes)
+			(show_name no)
+			(do_not_autoplace no)
+			(effects
+				(font
+					(size 1.27 1.27)
+				)
+			)
+		)
 		(pin "2"
 		)
@@
 			)
 		)
+		(property "MPN" "0402WGJ0103TCE"
+			(at 57.15 87.63 0)
+			(hide yes)
+			(show_name no)
+			(do_not_autoplace no)
+			(effects
+				(font
+					(size 1.27 1.27)
+				)
+			)
+		)
 		(pin "2"
 		)
@@
 			)
 		)
+		(property "MPN" "MAX3485ESA(UMW)"
+			(at 80.01 102.87 0)
+			(hide yes)
+			(show_name no)
+			(do_not_autoplace no)
+			(effects
+				(font
+					(size 1.27 1.27)
+				)
+			)
+		)
 		(pin "2"
 		)
@@
 			)
 		)
+		(property "MPN" ""
+			(at 163.83 96.52 0)
+			(hide yes)
+			(show_name no)
+			(do_not_autoplace no)
+			(effects
+				(font
+					(size 1.27 1.27)
+				)
+			)
+		)
 		(pin "1"
 		)
@@
 			)
 		)
+		(property "MPN" "0402WGJ0103TCE"
+			(at 41.91 34.29 0)
+			(hide yes)
+			(show_name no)
+			(do_not_autoplace no)
+			(effects
+				(font
+					(size 1.27 1.27)
+				)
+			)
+		)
 		(pin "1"
 		)
@@
 			)
 		)
+		(property "MPN" "0402WGF1200TCE"
+			(at 137.16 44.45 0)
+			(hide yes)
+			(show_name no)
+			(do_not_autoplace no)
+			(effects
+				(font
+					(size 1.27 1.27)
+				)
+			)
+		)
 		(pin "2"
 		)
@@
 			)
 		)
+		(property "MPN" "0402WGJ0103TCE"
+			(at 96.52 87.63 0)
+			(hide yes)
+			(show_name no)
+			(do_not_autoplace no)
+			(effects
+				(font
+					(size 1.27 1.27)
+				)
+			)
+		)
 		(pin "2"
 		)
@@
 			)
 		)
+		(property "MPN" "SM712"
+			(at 121.92 44.45 90)
+			(hide yes)
+			(show_name no)
+			(do_not_autoplace no)
+			(effects
+				(font
+					(size 1.27 1.27)
+				)
+			)
+		)
 		(pin "1"
 		)
@@
 			(at 41.91 87.63 0)
 			(hide yes)
+			(show_name no)
+			(do_not_autoplace no)
+			(effects
+				(font
+					(size 1.27 1.27)
+				)
+			)
+		)
+		(property "MPN" "0402WGJ0103TCE"
+			(at 41.91 87.63 0)
+			(hide yes)

Commit message: Autosave
Parts:
- added Q1: 2N7002, Package_TO_SOT_SMD:SOT-23, symbol Transistor_FET:2N7002
- added R43: 10k, Resistor_SMD:R_0402_1005Metric, symbol Device:R
- added R44: 33, Resistor_SMD:R_0402_1005Metric, symbol Device:R
- added U2: LTV-817S, Package_DIP:SMDIP-4_W9.53mm, symbol Isolator:LTV-817S
Connections:
- new net: R43.1, R44.1, U2.3
- new net: Q1.1 (G), R44.2
- new net +12V: U2.4
- new net GND1: Q1.2 (S), R43.2

Commit message: Autosave
Parts:
- added D1: US1M, Diode_SMD:D_SMA, symbol Diode:US1M
- added J6: p2r-05p, symbol joelib:p2r-05p
Connections:
- net +12V: now also D1.1 (K), J6.2 (coil_pos)
- net at Q1.3 (D): now also D1.2 (A), J6.1 (coil_neg)
