File: ETH.kicad_sch (KiCad schematic)
At the start: 34 parts, among them J5 https://abracon.com/Magnetics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, U3 LAN8742A, U4 USBLC6-4SC6, X1 NX2016SA-25.000M-STD-CZS-2

Commit message: Autosave
Parts:
- J5, U4: now fitted
Changed lines of the file:
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@@
 		(on_board yes)
 		(in_pos_files yes)
-		(dnp yes)
+		(dnp no)
 		(fields_autoplaced yes)
 		(property "Reference" "J5"
@@
 		(on_board yes)
 		(in_pos_files yes)
-		(dnp yes)
+		(dnp no)
 		(property "Reference" "U4"
 			(at 189.23 90.17 0)

Commit message: asf
Connections:
- net Earth: now also J5.8 (NC); no longer J5.SH
Changed lines of the file:
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@@
 		(pin "1"
 		)
-		(pin "SH"
+		(pin "8"
 		)
 		(pin "10"

Commit message: Autosave
Connections:
- net Earth: now also J5.SH; no longer J5.8 (NC)
Changed lines of the file:
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@@
 		(pin "1"
 		)
-		(pin "8"
+		(pin "SH"
 		)
 		(pin "10"

Commit message: Autosave
Parts:
- C21: MPN (none) -> 0402B471K500NT
- C22: MPN (none) -> CC0603KRX5R8BB105
- C23, C24, C25, C27: MPN (none) -> 0402F104M500NT
- C26: MPN (none) -> CL05A106MQ5NUNC
- C28, C29: MPN (none) -> 0402CG5R6C500NT
- C30: MPN (none) -> 0402B223K500NT
- C31: MPN (none) -> CC1206KKX7RDBB102
- L2: MPN (none) -> MCL2012S1R0MT
- R10, R14, R15, R16, R19, R22: MPN (none) -> 0402WGJ0103TCE
- R11, R12, R13, R18: MPN (none) -> 0402WGF330JTCE
- R17: MPN (none) -> 0402WGF1501TCE
- R20, R21: MPN (none) -> RTT022700FTH
- R5: MPN (none) -> 0402WGF1212TCE
- R6, R7, R8, R9: MPN (none) -> AC0402JR-0750RL
- U3: MPN (none) -> LAN8742AI-CZ-TR
- X1: MPN (none) -> NX2016SA-25MHZ-STD-CZS-2

Commit message: Autosave
Changed lines of the file:
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@@
 	)
 	(junction
+		(at 120.65 76.2)
+		(diameter 0)
+		(color 0 0 0 0)
+	)
+	(junction
 		(at 175.26 62.23)
 		(diameter 0)
@@
 	(wire
 		(pts
-			(xy 119.38 76.2) (xy 132.08 76.2)
+			(xy 119.38 76.2) (xy 120.65 76.2)
 		)
 		(stroke
@@
 	(wire
 		(pts
+			(xy 120.65 76.2) (xy 132.08 76.2)
+		)
+		(stroke
+			(width 0)
+			(type default)
+		)
+	)
+	(wire
+		(pts
 			(xy 201.93 130.81) (xy 191.77 130.81)
 		)
@@
 					(unit 1)
 				)
+			)
+		)
+	)
+	(symbol
+		(lib_id "power:PWR_FLAG")
+		(at 120.65 76.2 0)
+		(unit 1)
+		(body_style 1)
+		(exclude_from_sim no)
+		(in_bom yes)
+		(on_board yes)
+		(in_pos_files yes)
+		(dnp no)
+		(fields_autoplaced yes)
+		(property "Reference" "#FLG011"
+			(at 120.65 74.295 0)
+			(hide yes)
+			(show_name no)
+			(do_not_autoplace no)
+			(effects
+				(font
+					(size 1.27 1.27)
+				)
+			)
+		)
+		(property "Value" "PWR_FLAG"
+			(at 120.65 71.12 0)
+			(show_name no)
+			(do_not_autoplace no)
+			(effects
+				(font
+					(size 1.27 1.27)
+				)
+			)
+		)
+		(property "Footprint" ""
+			(at 120.65 76.2 0)
+			(hide yes)
+			(show_name no)
+			(do_not_autoplace no)
+			(effects
+				(font
+					(size 1.27 1.27)
+				)
+			)
+		)
+		(property "Datasheet" ""
+			(at 120.65 76.2 0)
+			(hide yes)
+			(show_name no)
+			(do_not_autoplace no)
+			(effects
+				(font
+					(size 1.27 1.27)
+				)
+			)
+		)
+		(property "Description" "Special symbol for telling ERC where power comes from"
+			(at 120.65 76.2 0)
+			(hide yes)
+			(show_name no)
+			(do_not_autoplace no)
+			(effects
+				(font
+					(size 1.27 1.27)
+				)
+			)
+		)
+		(pin "1"
+		)
+		(instances
+			(project "mainbrd3"
+				(path "/89e0f049-91ab-4c37-b514-d5ee0e775d39/fa672b14-329a-4bb7-a909-5b1dde7a1a04"
+					(reference "#FLG011")
+					(unit 1)
+				)

Commit message: Autosave
Connections:
- net Earth renamed Shield_Island
Changed lines of the file:
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@@
-	)
-	(symbol
-		(lib_id "power:Earth")
-		(at 242.57 144.78 0)
-		(unit 1)
-		(body_style 1)
-		(exclude_from_sim no)
-		(in_bom yes)
-		(on_board yes)
-		(in_pos_files yes)
-		(dnp no)
-		(fields_autoplaced yes)
-		(property "Reference" "#PWR056"
-			(at 242.57 151.13 0)
-			(hide yes)
-			(show_name no)
-			(do_not_autoplace no)
-			(effects
-				(font
-					(size 1.27 1.27)
-				)
-			)
-		)
-		(property "Value" "Earth"
-			(at 242.57 149.86 0)
-			(show_name no)
-			(do_not_autoplace no)
-			(effects
-				(font
-					(size 1.27 1.27)
-				)
-			)
-		)
-		(property "Footprint" ""
-			(at 242.57 144.78 0)
-			(hide yes)
-			(show_name no)
-			(do_not_autoplace no)
-			(effects
-				(font
-					(size 1.27 1.27)
-				)
-			)
-		)
-		(property "Datasheet" ""
-			(at 242.57 144.78 0)
-			(hide yes)
-			(show_name no)
-			(do_not_autoplace no)
-			(effects
-				(font
-					(size 1.27 1.27)
-				)
-			)
-		)
-		(property "Description" "Power symbol creates a global label with name \"Earth\""
-			(at 242.57 144.78 0)
-			(hide yes)
-			(show_name no)
-			(do_not_autoplace no)
-			(effects
-				(font
-					(size 1.27 1.27)
-				)
-			)
-		)
-		(pin "1"
-		)
-		(instances
-			(project "mainbrd3"
-				(path "/89e0f049-91ab-4c37-b514-d5ee0e775d39/fa672b14-329a-4bb7-a909-5b1dde7a1a04"
-					(reference "#PWR056")
-					(unit 1)
-				)
-			)
-		)
 	)
 	(symbol
@@
 					(unit 1)
 				)
+			)
+		)
+	)
+	(symbol
+		(lib_id "power:Earth")
+		(at 242.57 144.78 0)
+		(unit 1)
+		(body_style 1)
+		(exclude_from_sim no)
+		(in_bom yes)
+		(on_board yes)
+		(in_pos_files yes)
+		(dnp no)
+		(fields_autoplaced yes)
+		(property "Reference" "#PWR076"
+			(at 242.57 151.13 0)
+			(hide yes)
+			(show_name no)
+			(do_not_autoplace no)
+			(effects
+				(font
+					(size 1.27 1.27)
+				)
+			)
+		)
+		(property "Value" "Shield_Island"
+			(at 242.57 149.86 0)
+			(show_name no)
+			(do_not_autoplace no)
+			(effects
+				(font
+					(size 1.27 1.27)
+				)
+			)
+		)
+		(property "Footprint" ""
+			(at 242.57 144.78 0)
+			(hide yes)
+			(show_name no)
+			(do_not_autoplace no)
+			(effects
+				(font
+					(size 1.27 1.27)
+				)
+			)
+		)
+		(property "Datasheet" ""
+			(at 242.57 144.78 0)
+			(hide yes)
+			(show_name no)
+			(do_not_autoplace no)
+			(effects
+				(font
+					(size 1.27 1.27)
+				)
+			)
+		)
+		(property "Description" "Power symbol creates a global label with name \"Earth\""
+			(at 242.57 144.78 0)
+			(hide yes)
+			(show_name no)
+			(do_not_autoplace no)
+			(effects
+				(font
+					(size 1.27 1.27)
+				)
+			)
+		)
+		(pin "1"
+		)
+		(instances
+			(project "mainbrd3"
+				(path "/89e0f049-91ab-4c37-b514-d5ee0e775d39/fa672b14-329a-4bb7-a909-5b1dde7a1a04"
+					(reference "#PWR076")
+					(unit 1)
+				)

Commit message: abc
Connections:
- net Shield_Island: now also J5.8 (NC); no longer J5.SH
Changed lines of the file:
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@@
 		(pin "1"
 		)
-		(pin "SH"
+		(pin "8"
 		)
 		(pin "10"
